File: AlarmClock/AlarmClock.sch (KiCad schematic (older format))
At the start: 39 parts, among them Q1 2N3904, Q2 2N3904, Q3 2N3904, Q4 2N3904, Q5 2N3904, SW1 SW_Push, SW2 SW_Push, SW3 SW_Push, SW4 SW_Push, SW5 SW_Push, U1 LM386, U2 LTC-4727JR, U3 LM358

Commit message: updated
Parts:
- removed D1: Diode, ECE:DO41, symbol Diode
- R16: value 200Ω -> 30Ω
- renumbered D2 to D1
Connections:
- net +3V3: no longer STM1.2-5 (3V), STM1.2-6 (3V), U3.8 (V+)
- net at C2.2 (-): now also LS1.1
- net +5VD: now reaches STM1.2-3 (5V)
- no-connect marks 70 -> 69
Changed lines of the file:
@@
-	1    0    0    -1
-$EndComp
-$Comp
-L STM32_F4 STM1
-U 1 1 5B2807A9
-P 5900 3750
-F 0 "STM1" H 5900 3850 60  0000 C CNN
-F 1 "STM32_F407" H 5900 3650 60  0000 C CNN
-F 2 "ECE:STM32_F4" H 5900 3750 60  0001 C CNN
-F 3 "" H 5900 3750 60  0000 C CNN
-	1    5900 3750
 	1    0    0    -1
 $EndComp
@@
 NoConn ~ 4900 1400
 $Comp
-L +3.3V #PWR08
-U 1 1 5B2BF7FF
-P 6300 1050
-F 0 "#PWR08" H 6300 900 50  0001 C CNN
-F 1 "+3.3V" H 6425 1050 50  0000 C CNN
-F 2 "" H 6300 1050 50  0001 C CNN
-F 3 "" H 6300 1050 50  0001 C CNN
-	1    6300 1050
-	1    0    0    -1
-$EndComp
-$Comp
 L +5V #PWR09
 U 1 1 5B2BF88B
@@
 NoConn ~ 5600 1050
 NoConn ~ 5700 1050
-NoConn ~ 5900 1050
 $Comp
 L CAP_POL C4
@@
 	1    0    0    -1
 $EndComp
-$Comp
-L +3.3V #PWR014
-U 1 1 5B36C086
-P 10050 1300
-F 0 "#PWR014" H 10050 1150 50  0001 C CNN
-F 1 "+3.3V" H 10050 1440 50  0000 C CNN
-F 2 "" H 10050 1300 50  0001 C CNN
-F 3 "" H 10050 1300 50  0001 C CNN
-	1    10050 1300
-	1    0    0    -1
-$EndComp
 Text GLabel 8150 1600 0    60   Input ~ 0
 PA4
@@
 P 2600 1900
 F 0 "R16" H 2600 2075 40  0000 C CNN
-F 1 "200Ω" H 2600 2000 40  0000 C CNN
+F 1 "30Ω" H 2600 2000 40  0000 C CNN
 F 2 "ECE:RES.3" H 2600 1970 30  0001 C CNN
 F 3 "" V 2600 1900 30  0000 C CNN
 	1    2600 1900
 	-1   0    0    1
-$EndComp
-$Comp
-L +3V3 #PWR015
-U 1 1 5B3BF19D
-P 6200 1050
-F 0 "#PWR015" H 6200 900 50  0001 C CNN
-F 1 "+3V3" H 6200 1190 50  0000 C CNN
-F 2 "" H 6200 1050 50  0001 C CNN
-F 3 "" H 6200 1050 50  0001 C CNN
-	1    6200 1050
-	1    0    0    -1
-$EndComp
-$Comp
-L +3V3 #PWR016
-U 1 1 5B3BFF09
-P 10050 3000
-F 0 "#PWR016" H 10050 2850 50  0001 C CNN
-F 1 "+3V3" H 10050 3140 50  0000 C CNN
-F 2 "" H 10050 3000 50  0001 C CNN
-F 3 "" H 10050 3000 50  0001 C CNN
-	1    10050 3000
-	1    0    0    -1
 $EndComp
 Text GLabel 8475 3475 0    60   Input ~ 0
@@
 Text GLabel 8525 5550 0    60   Input ~ 0
 PC11
+$Comp
+L SW_Push SW1
+U 1 1 5B3C2F2D
+P 9275 3475
+F 0 "SW1" H 9325 3575 50  0000 L CNN
+F 1 "SW_Push" H 9275 3415 50  0000 C CNN
+F 2 "Buttons_Switches_THT:SW_PUSH_6mm" H 9275 3675 50  0001 C CNN
+F 3 "" H 9275 3675 50  0001 C CNN
+	1    9275 3475
+	1    0    0    -1
+$EndComp
+$Comp
+L SW_Push SW2
+U 1 1 5B3C2FB8
+P 9275 4000
+F 0 "SW2" H 9325 4100 50  0000 L CNN
+F 1 "SW_Push" H 9275 3940 50  0000 C CNN
+F 2 "Buttons_Switches_THT:SW_PUSH_6mm" H 9275 4200 50  0001 C CNN
+F 3 "" H 9275 4200 50  0001 C CNN
+	1    9275 4000
+	1    0    0    -1
+$EndComp
+$Comp
+L SW_Push SW3
+U 1 1 5B3C301B
+P 9275 4525
+F 0 "SW3" H 9325 4625 50  0000 L CNN
+F 1 "SW_Push" H 9275 4465 50  0000 C CNN
+F 2 "Buttons_Switches_THT:SW_PUSH_6mm" H 9275 4725 50  0001 C CNN
+F 3 "" H 9275 4725 50  0001 C CNN
+	1    9275 4525
+	1    0    0    -1
+$EndComp
+$Comp
+L SW_Push SW4
+U 1 1 5B3C30A4
+P 9275 5050
+F 0 "SW4" H 9325 5150 50  0000 L CNN
+F 1 "SW_Push" H 9275 4990 50  0000 C CNN
+F 2 "Buttons_Switches_THT:SW_PUSH_6mm" H 9275 5250 50  0001 C CNN
+F 3 "" H 9275 5250 50  0001 C CNN
+	1    9275 5050
+	1    0    0    -1
+$EndComp
+$Comp
+L SW_Push SW5
+U 1 1 5B3C3113
+P 9275 5550
+F 0 "SW5" H 9325 5650 50  0000 L CNN
+F 1 "SW_Push" H 9275 5490 50  0000 C CNN
+F 2 "Buttons_Switches_THT:SW_PUSH_6mm" H 9275 5750 50  0001 C CNN
+F 3 "" H 9275 5750 50  0001 C CNN
+	1    9275 5550
+	1    0    0    -1
+$EndComp
 Wire Wire Line
 	1750 2000 1550 2000
@@
 Wire Wire Line
 	9075 3475 8475 3475
+Wire Wire Line
+	3350 1900 3700 1900
+Wire Wire Line
+	10050 3000 10050 3150
+Wire Wire Line
+	10050 3450 10050 5550
+Connection ~ 10350 1700
+Connection ~ 1850 1350
+Connection ~ 8650 1600
+$Comp
+L +3V3 #PWR016
+U 1 1 5B3BFF09
+P 10050 3000
+F 0 "#PWR016" H 10050 2850 50  0001 C CNN
+F 1 "+3V3" H 10050 3140 50  0000 C CNN
+F 2 "" H 10050 3000 50  0001 C CNN
+F 3 "" H 10050 3000 50  0001 C CNN
+	1    10050 3000
+	1    0    0    -1
+$EndComp
 $Comp
 L Diode D1
-U 1 1 5B3C0B12
-P 3500 1900
-F 0 "D1" H 3500 2000 50  0000 C CNN
-F 1 "Diode" H 3500 1800 50  0000 C CNN
-F 2 "ECE:DO41" H 3500 1900 50  0000 C CNN
-F 3 "" H 3500 1900 50  0000 C CNN
-	1    3500 1900
-	-1   0    0    1
-$EndComp
-Wire Wire Line
-	3700 1900 3650 1900
-$Comp
-L Diode D2
 U 1 1 5B3C12E0
 P 10050 3300
-F 0 "D2" H 10050 3400 50  0000 C CNN
+F 0 "D1" H 10050 3400 50  0000 C CNN
 F 1 "Diode" H 10050 3200 50  0000 C CNN
 F 2 "ECE:DO41" H 10050 3300 50  0000 C CNN
@@
 	0    -1   -1   0
 $EndComp
-Wire Wire Line
-	10050 3000 10050 3150
-Wire Wire Line
-	10050 3450 10050 5550
-Connection ~ 10350 1700
-Connection ~ 1850 1350
-$Comp
-L SW_Push SW1
-U 1 1 5B3C2F2D
-P 9275 3475
-F 0 "SW1" H 9325 3575 50  0000 L CNN
-F 1 "SW_Push" H 9275 3415 50  0000 C CNN
-F 2 "Buttons_Switches_THT:SW_PUSH_6mm" H 9275 3675 50  0001 C CNN
-F 3 "" H 9275 3675 50  0001 C CNN
-	1    9275 3475
-	1    0    0    -1
-$EndComp
-$Comp
-L SW_Push SW2
-U 1 1 5B3C2FB8
-P 9275 4000
-F 0 "SW2" H 9325 4100 50  0000 L CNN
-F 1 "SW_Push" H 9275 3940 50  0000 C CNN
-F 2 "Buttons_Switches_THT:SW_PUSH_6mm" H 9275 4200 50  0001 C CNN
-F 3 "" H 9275 4200 50  0001 C CNN
-	1    9275 4000
-	1    0    0    -1
-$EndComp
-$Comp
-L SW_Push SW3
-U 1 1 5B3C301B
-P 9275 4525
-F 0 "SW3" H 9325 4625 50  0000 L CNN
-F 1 "SW_Push" H 9275 4465 50  0000 C CNN
-F 2 "Buttons_Switches_THT:SW_PUSH_6mm" H 9275 4725 50  0001 C CNN
-F 3 "" H 9275 4725 50  0001 C CNN
-	1    9275 4525
-	1    0    0    -1
-$EndComp
-$Comp
-L SW_Push SW4
-U 1 1 5B3C30A4
-P 9275 5050
-F 0 "SW4" H 9325 5150 50  0000 L CNN
-F 1 "SW_Push" H 9275 4990 50  0000 C CNN
-F 2 "Buttons_Switches_THT:SW_PUSH_6mm" H 9275 5250 50  0001 C CNN
-F 3 "" H 9275 5250 50  0001 C CNN
-	1    9275 5050
-	1    0    0    -1
-$EndComp
-$Comp
-L SW_Push SW5
-U 1 1 5B3C3113
-P 9275 5550
-F 0 "SW5" H 9325 5650 50  0000 L CNN
-F 1 "SW_Push" H 9275 5490 50  0000 C CNN
-F 2 "Buttons_Switches_THT:SW_PUSH_6mm" H 9275 5750 50  0001 C CNN
-F 3 "" H 9275 5750 50  0001 C CNN
-	1    9275 5550
-	1    0    0    -1
-$EndComp
-Connection ~ 8650 1600
+$Comp
+L STM32_F4 STM1
+U 1 1 5B2807A9
+P 5900 3750
+F 0 "STM1" H 5900 3850 60  0000 C CNN
+F 1 "STM32_F407" H 5900 3650 60  0000 C CNN
+F 2 "ECE:STM32_F4" H 5900 3750 60  0001 C CNN
+F 3 "" H 5900 3750 60  0000 C CNN
+	1    5900 3750
+	1    0    0    -1
+$EndComp
+$Comp
+L +5VD #PWR?
+U 1 1 5B767456
+P 5900 1050
+F 0 "#PWR?" H 5900 900 50  0001 C CNN
+F 1 "+5VD" H 5900 1190 50  0000 C CNN
+F 2 "" H 5900 1050 50  0001 C CNN
+F 3 "" H 5900 1050 50  0001 C CNN
+	1    5900 1050
+	1    0    0    -1
+$EndComp
+$Comp
+L +5VD #PWR?
+U 1 1 5B76759A
+P 10050 1275
+F 0 "#PWR?" H 10050 1125 50  0001 C CNN
+F 1 "+5VD" H 10050 1415 50  0000 C CNN
+F 2 "" H 10050 1275 50  0001 C CNN
+F 3 "" H 10050 1275 50  0001 C CNN
+	1    10050 1275
+	1    0    0    -1
+$EndComp
 $EndSCHEMATC
